Commit message: Changed orientation of eef to match open rave test orientation

File: katana_description/urdf/katana_300_6m180.urdf.xacro (robot description, xacro)
@@ -212,4 +212,14 @@
       </inertial>
     </link>
+	    <joint name="katana_gripper_atool_frame_joint" type="fixed">
+      <parent link="katana_motor5_wrist_roll_link"/>
+      <child link="katana_gripper_atool_frame_joint" />
+      <origin xyz="0 0 -${link5_length}" rpy="${-M_PI/2} 0 ${M_PI/2}"/>
+    </joint>
+    <link name="katana_gripper_atool_frame_joint">
+      <!-- This is the coordinate system of the tool (this is the position
+         used in IK etc., relative to the base frame); there is no actual
+         arm part attached to this link -->
+  </link>
     <joint name="katana_gripper_joint" type="fixed">
       <parent link="katana_motor5_wrist_roll_link" />
@@ -271,23 +281,3 @@
     <xacro:finger prefix="r" rotate="0" />
     <xacro:finger prefix="l" rotate="${M_PI}" />
-    <joint name="katana_gripper_tool_frame_joint" type="fixed">
-      <parent link="katana_motor5_wrist_roll_link"/>
-      <child link="katana_gripper_tool_frame" />
-      <origin xyz="0 0 -${link5_length}" rpy="0 ${M_PI/2} 0"/>
-    </joint>
-    <link name="katana_gripper_tool_frame">
-      <!-- This is the coordinate system of the tool (this is the position
-         used in IK etc., relative to the base frame); there is no actual
-         arm part attached to this link -->
-  </link>
-  <!-- **************************************************************** -->
-  <joint name="katana_base_frame_joint" type="fixed">
-    <parent link="katana_base_link"/>
-    <child link="katana_base_frame" />
-    <origin xyz="0 0 ${base_height}" rpy="0 0 0"/>
-  </joint>
-  <link name="katana_base_frame">
-    <!-- This is the reference coordinate system of the arm (the KNI kinematics are specified
-         in this frame); there is no actual arm part attached to this link -->
-  </link>
 </robot>

Commit message: reverted to standard urdf

File: katana_description/urdf/katana_300_6m180.urdf.xacro (robot description, xacro)
@@ -212,14 +212,4 @@
       </inertial>
     </link>
-	    <joint name="katana_gripper_atool_frame_joint" type="fixed">
-      <parent link="katana_motor5_wrist_roll_link"/>
-      <child link="katana_gripper_atool_frame_joint" />
-      <origin xyz="0 0 -${link5_length}" rpy="${-M_PI/2} 0 ${M_PI/2}"/>
-    </joint>
-    <link name="katana_gripper_atool_frame_joint">
-      <!-- This is the coordinate system of the tool (this is the position
-         used in IK etc., relative to the base frame); there is no actual
-         arm part attached to this link -->
-  </link>
     <joint name="katana_gripper_joint" type="fixed">
       <parent link="katana_motor5_wrist_roll_link" />
@@ -281,3 +271,23 @@
     <xacro:finger prefix="r" rotate="0" />
     <xacro:finger prefix="l" rotate="${M_PI}" />
+    <joint name="katana_gripper_tool_frame_joint" type="fixed">
+      <parent link="katana_motor5_wrist_roll_link"/>
+      <child link="katana_gripper_tool_frame" />
+      <origin xyz="0 0 -${link5_length}" rpy="0 ${M_PI/2} 0"/>
+    </joint>
+    <link name="katana_gripper_tool_frame">
+      <!-- This is the coordinate system of the tool (this is the position
+         used in IK etc., relative to the base frame); there is no actual
+         arm part attached to this link -->
+  </link>
+  <!-- **************************************************************** -->
+  <joint name="katana_base_frame_joint" type="fixed">
+    <parent link="katana_base_link"/>
+    <child link="katana_base_frame" />
+    <origin xyz="0 0 ${base_height}" rpy="0 0 0"/>
+  </joint>
+  <link name="katana_base_frame">
+    <!-- This is the reference coordinate system of the arm (the KNI kinematics are specified
+         in this frame); there is no actual arm part attached to this link -->
+  </link>
 </robot>

Commit message: Changed urdf for moveit and ikfast

File: katana_description/urdf/katana_300_6m180.urdf.xacro (robot description, xacro)
@@ -14,4 +14,5 @@
   <property name="link4_length" value="0.1523" />
   <property name="link5_length" value="0.1505" />
+  <property name="tool_frame_offset" value="-0.11" />
   <!-- All inertial values (mass, center of mass and inertia tensor) have been
        calculated from the meshes using MeshLab -->
@@ -274,5 +275,5 @@
       <parent link="katana_motor5_wrist_roll_link"/>
       <child link="katana_gripper_tool_frame" />
-      <origin xyz="0 0 -${link5_length}" rpy="0 ${M_PI/2} 0"/>
+      <origin xyz="0 0 ${tool_frame_offset}" rpy="0 ${M_PI/2} 0"/>
     </joint>
     <link name="katana_gripper_tool_frame">
@@ -281,13 +282,3 @@
          arm part attached to this link -->
   </link>
-  <!-- **************************************************************** -->
-  <joint name="katana_base_frame_joint" type="fixed">
-    <parent link="katana_base_link"/>
-    <child link="katana_base_frame" />
-    <origin xyz="0 0 ${base_height}" rpy="0 0 0"/>
-  </joint>
-  <link name="katana_base_frame">
-    <!-- This is the reference coordinate system of the arm (the KNI kinematics are specified
-         in this frame); there is no actual arm part attached to this link -->
-  </link>
 </robot>

Commit message: Changed urdf for moveit and ikfast

File: katana_description/urdf/katana_300_6m180.urdf.xacro (robot description, xacro)
@@ -14,4 +14,5 @@
   <property name="link4_length" value="0.1523" />
   <property name="link5_length" value="0.1505" />
+  <property name="tool_frame_offset" value="-0.11" />
   <!-- All inertial values (mass, center of mass and inertia tensor) have been
        calculated from the meshes using MeshLab -->
@@ -318,5 +319,5 @@
       <parent link="katana_motor5_wrist_roll_link"/>
       <child link="katana_gripper_tool_frame" />
-      <origin xyz="0 0 -${link5_length}" rpy="0 ${M_PI/2} 0"/>
+      <origin xyz="0 0 ${tool_frame_offset}" rpy="0 ${M_PI/2} 0"/>
     </joint>
     <link name="katana_gripper_tool_frame">
@@ -325,13 +326,3 @@
          arm part attached to this link -->
   </link>
-  <!-- **************************************************************** -->
-  <joint name="katana_base_frame_joint" type="fixed">
-    <parent link="katana_base_link"/>
-    <child link="katana_base_frame" />
-    <origin xyz="0 0 ${base_height}" rpy="0 0 0"/>
-  </joint>
-  <link name="katana_base_frame">
-    <!-- This is the reference coordinate system of the arm (the KNI kinematics are specified
-         in this frame); there is no actual arm part attached to this link -->
-  </link>
 </robot>

Commit message: Added the distance discs to the katana wrist link

File: katana_description/urdf/katana_300_6m180.urdf.xacro (robot description, xacro)
@@ -212,4 +212,25 @@
       </inertial>
     </link>
+	<joint name="katana_motor5_wrist_roll_discs_joint" type="fixed">
+      <parent link="katana_motor5_wrist_roll_link" />
+      <child link="katana_motor5_wrist_roll_discs" />
+      <origin rpy="0 ${M_PI/2} 0" xyz="0.0375 0 0"/>
+    </joint>
+    <link name="katana_motor5_wrist_roll_discs">
+    <visual>
+      <origin xyz="0 0 0" rpy="0 0 0" />
+      <geometry>
+        <cylinder length="0.025" radius="0.025" />
+      </geometry>
+      <material name="grey" />
+    </visual>
+    <collision>
+      <origin xyz="0 0 0" rpy="0 0 0" />
+      <geometry>
+        <cylinder length="0.025" radius="0.025" />
+      </geometry>
+    </collision>
+    <xacro:cylinder_inertial length="0.025" radius="0.025"  mass="0.05" />
+  </link>
     <joint name="katana_gripper_joint" type="fixed">
       <parent link="katana_motor5_wrist_roll_link" />

Commit message: Added the distance discs to the katana wrist link

File: katana_description/urdf/katana_300_6m180.urdf.xacro (robot description, xacro)
@@ -213,4 +213,25 @@
       </inertial>
     </link>
+	<joint name="katana_motor5_wrist_roll_discs_joint" type="fixed">
+      <parent link="katana_motor5_wrist_roll_link" />
+      <child link="katana_motor5_wrist_roll_discs" />
+      <origin rpy="0 ${M_PI/2} 0" xyz="0.0375 0 0"/>
+    </joint>
+    <link name="katana_motor5_wrist_roll_discs">
+    <visual>
+      <origin xyz="0 0 0" rpy="0 0 0" />
+      <geometry>
+        <cylinder length="0.025" radius="0.025" />
+      </geometry>
+      <material name="grey" />
+    </visual>
+    <collision>
+      <origin xyz="0 0 0" rpy="0 0 0" />
+      <geometry>
+        <cylinder length="0.025" radius="0.025" />
+      </geometry>
+    </collision>
+    <xacro:cylinder_inertial length="0.025" radius="0.025"  mass="0.05" />
+  </link>
     <joint name="katana_gripper_joint" type="fixed">
       <parent link="katana_motor5_wrist_roll_link" />

Commit message: Changed finger orientation to match our real Katana's gripper.

File: katana_description/urdf/katana_300_6m180.urdf.xacro (robot description, xacro)
@@ -248,5 +248,5 @@
       <link name="katana_${prefix}_finger_link">
         <visual>
-          <origin rpy="0 ${M_PI} 0" xyz="0 0 0"/>
+          <origin rpy="0 ${M_PI} 0.27" xyz="0 0 0"/>
           <geometry>
             <mesh filename="package://katana_description/meshes/katana/katana_gripper_${prefix}_finger.stl"/>
@@ -255,5 +255,5 @@
         </visual>
         <collision>
-          <origin rpy="0 ${M_PI} 0" xyz="0 0 0"/>
+          <origin rpy="0 ${M_PI} 0.27" xyz="0 0 0"/>
           <geometry>
             <mesh filename="package://katana_description/meshes/katana/convex/katana_gripper_${prefix}_finger_convex.stl"/>
@@ -268,4 +268,27 @@
         </inertial>
       </link>
+      <!--
+      <joint name="katana__${prefix}_finger_tip_join" type="fixed">
+        <parent link="katana_${prefix}_finger_link" />
+        <child link="kurtana__${prefix}_finger_tip_link" />
+        <origin rpy="0 0 0.37" xyz="0.09 0.045 0"/>
+      </joint>
+      <link name="kurtana__${prefix}_finger_tip_link">
+	    <visual>
+	      <origin xyz="0 0 0" rpy="0 0 0" />
+	      <geometry>
+	        <box size="0.02 0.005 0.02" />
+	      </geometry>
+	      <material name="grey" />
+	    </visual>
+	    <collision>
+	      <origin xyz="0 0 0" rpy="0 0 0" />
+	      <geometry>
+	        <box size="0.02 0.005 0.02" />
+	      </geometry>
+	    </collision>
+	    <xacro:box_inertial x="0.02" y="0.005" z="0.02" mass="0.01" />
+	  </link>
+	  -->
     </xacro:macro>
     <xacro:finger prefix="r" rotate="0" />

Commit message: Changed finger orientation to match our real Katana's gripper.

File: katana_description/urdf/katana_300_6m180.urdf.xacro (robot description, xacro)
@@ -270,5 +270,5 @@
       <link name="katana_${prefix}_finger_link">
         <visual>
-          <origin rpy="0 ${M_PI} 0" xyz="0 0 0"/>
+          <origin rpy="0 ${M_PI} 0.27" xyz="0 0 0"/>
           <geometry>
             <mesh filename="package://katana_description/meshes/katana/katana_gripper_${prefix}_finger.stl"/>
@@ -277,5 +277,5 @@
         </visual>
         <collision>
-          <origin rpy="0 ${M_PI} 0" xyz="0 0 0"/>
+          <origin rpy="0 ${M_PI} 0.27" xyz="0 0 0"/>
           <geometry>
             <mesh filename="package://katana_description/meshes/katana/convex/katana_gripper_${prefix}_finger_convex.stl"/>
@@ -290,4 +290,27 @@
         </inertial>
       </link>
+      <!--
+      <joint name="katana__${prefix}_finger_tip_join" type="fixed">
+        <parent link="katana_${prefix}_finger_link" />
+        <child link="kurtana__${prefix}_finger_tip_link" />
+        <origin rpy="0 0 0.37" xyz="0.09 0.045 0"/>
+      </joint>
+      <link name="kurtana__${prefix}_finger_tip_link">
+	    <visual>
+	      <origin xyz="0 0 0" rpy="0 0 0" />
+	      <geometry>
+	        <box size="0.02 0.005 0.02" />
+	      </geometry>
+	      <material name="grey" />
+	    </visual>
+	    <collision>
+	      <origin xyz="0 0 0" rpy="0 0 0" />
+	      <geometry>
+	        <box size="0.02 0.005 0.02" />
+	      </geometry>
+	    </collision>
+	    <xacro:box_inertial x="0.02" y="0.005" z="0.02" mass="0.01" />
+	  </link>
+	  -->
     </xacro:macro>
     <xacro:finger prefix="r" rotate="0" />

Commit message: Try to make gripper faster

File: katana_description/urdf/katana_300_6m180.urdf.xacro (robot description, xacro)
@@ -266,5 +266,5 @@
         <origin rpy="${rotate} 0 0" xyz="0.034 0 0"/>
         <axis xyz="0 0 1"/>
-        <limit effort="0.5" lower="-0.44" upper="0.30"  velocity="0.718834"/>
+        <limit effort="0.5" lower="-0.85" upper="0.30"  velocity="1"/>
       </joint>
       <link name="katana_${prefix}_finger_link">
